File: esp32c3_sim7600/esp32c3.kicad_sch (KiCad schematic)
At the start: 10 parts, among them J1 Conn_01x04_Socket, J2 Conn_01x04_Socket, SW1 SW_Push, SW2 SW_Push, U1 ESP32-C3-MINI-1-N4

Commit message: completed routing
Parts:
- removed J1, J2: Conn_01x04_Socket, Connector_PinHeader_2.54mm:PinHeader_1x04_P2.54mm_Vertical, symbol Connector:Conn_01x04_Socket
- added J8, J9: Conn_01x06_Pin, Connector_PinHeader_2.54mm:PinHeader_1x06_P2.54mm_Vertical, symbol Connector:Conn_01x06_Pin
- SW1, SW2: footprint Button_Switch_THT:SW_PUSH_6mm -> Button_Switch_SMD:SW_Push_1P1T_NO_CK_KMR2
Connections:
- net 3V3: now also J8.1 (Pin_1), J9.1 (Pin_1)
- net GND: now also J8.2 (Pin_2), J9.2 (Pin_2)
- net IO0: now also J8.5 (Pin_5)
- net IO1: now also J8.6 (Pin_6)
- net IO2: now also J8.3 (Pin_3)
- net IO3: now also J8.4 (Pin_4)
- net IO4: now also J9.6 (Pin_6)
- net IO5: now also J9.5 (Pin_5)
- net IO6: now also J9.4 (Pin_4)
- net IO7: now also J9.3 (Pin_3)
