File: esp32c3_sim7600/sim7600.kicad_sch (KiCad schematic)
At the start: 48 parts, among them J4 CONUFL001-SMD-T, J5 CONUFL001-SMD-T, J6 CONUFL001-SMD-T, J7 SIM7050-6-0-00-X_REVC, Q1 NPN, Q2 NPN, Q3 NPN, U4 SIM7600E, U6 TXB0108RGY

Commit message: completed routing
Parts:
- removed R14, R15, R16, R17, R18, R19, R20, R21, R22, R23, R24, R25: 47K, Resistor_SMD:R_0603_1608Metric, symbol Device:R
Connections:
- net GND: now also U6.12 (B8), U6.13 (B7), U6.14 (B6), U6.15 (B5), U6.16 (B4), U6.17 (B3), U6.4 (A3), U6.5 (A4), U6.6 (A5), U6.7 (A6), U6.8 (A7), U6.9 (A8)
